Commit message: Update URDF xacro files

File: urdf/crx_gripper_gz_ros2_control_macro.xacro (robot description, xacro)
@@ -37,6 +37,17 @@
       </joint>
       <xacro:if value="${use_robotiq_gripper == True or use_robotiq_gripper == 'true'}">
-        <!-- Gazebo handles the mimic (right knuckle) natively; only the driven joint needs an interface. -->
+        <!-- Both jaws are driven explicitly (no mimic): DART ignores mimic constraints, so each
+             prismatic jaw needs its own command interface. A joint_trajectory_controller commands
+             both to the same position for symmetric parallel closing. -->
         <joint name="${prefix}robotiq_85_left_knuckle_joint">
+          <command_interface name="position"/>
+          <state_interface name="position">
+            <param name="initial_value">0.0</param>
+          </state_interface>
+          <state_interface name="velocity">
+            <param name="initial_value">0.0</param>
+          </state_interface>
+        </joint>
+        <joint name="${prefix}robotiq_85_right_knuckle_joint">
           <command_interface name="position"/>
           <state_interface name="position">

File: urdf/robotiq_2f_85_simple_parallel.urdf.xacro (robot description, xacro)
@@ -1,5 +1,6 @@
 <?xml version="1.0"?>
 <!-- Simplified Robotiq 2F-85 for Gazebo: two rigid jaws, parallel closing via prismatic joints from base
-     (ABB-like linear motion). One commanded joint + mimic on the other side. No inner knuckle chain.
+     (ABB-like linear motion). BOTH jaws are real command joints driven by a joint_trajectory_controller
+     (no <mimic>: DART/gz physics does not support mimic constraints, so the mimic'd jaw never moved).
      Stroke 0.043 m per finger (~85 mm opening between pads). Same link/joint names for ros2_control / MoveIt. -->
 <robot xmlns:xacro="http://wiki.ros.org/xacro" name="robotiq_gripper">
@@ -222,5 +223,4 @@
             <origin xyz="-0.03060114 0.0 0.05490452" rpy="0 0 0" />
             <limit lower="0.0" upper="${robotiq_prismatic_stroke}" effort="50" velocity="0.5" />
-            <mimic joint="${prefix}robotiq_85_left_knuckle_joint" multiplier="1" />
         </joint>
     </xacro:macro>
