Commit message: Fix gripper: both jaws real joints + DART limit-lock workaround
The Robotiq sim gripper could not grasp anything, for two stacked reasons:

1. The right jaw was a <mimic> joint, but DART (gz-sim default physics)
   does not support mimic constraints ("no constraint will be created"),
   so the right jaw was never actuated at all. Both jaws are now real,
   independently commanded prismatic joints driven together by a
   joint_trajectory_controller (gripper_controller, action
   /gripper_controller/follow_joint_trajectory).

2. Even as a real joint the lower jaw stayed frozen: DART locks a
   velocity-servo-driven joint whose limit constraint is engaged, and
   whichever jaw hangs below the horizontal gripper is pressed into its
   lower limit (q=0 = open) by gravity. Verified by rolling the wrist
   180 deg: the "dead" jaw started working and the "good" jaw froze.
   Fixed by giving the open pose margin from the limit (lower=-0.002)
   and adding 5 N Coulomb friction (> 1.3 N jaw weight) so an
   uncontrolled jaw never sags onto the limit in any pose.

Verified in the worst-case (home) pose: close moves both jaws 0.04
toward center, open returns both to start.

Co-Authored-By: Claude Fable 5 <noreply@anthropic.com>

File: urdf/robotiq_2f_85_simple_parallel.urdf.xacro (robot description, xacro)
@@ -209,5 +209,13 @@
             <xacro:insert_block name="origin" />
         </joint>
-        <!-- q=0: open; q=stroke: closed. Left jaw moves along -X toward center when q increases. -->
+        <!-- q=0: open; q=stroke: closed. Left jaw moves along -X toward center when q increases.
+             Two DART-specific guards on both jaw joints (found empirically; see git history):
+             - lower limit is -0.002 (not 0.0) so the commanded open pose q=0 sits INSIDE the
+               range: DART locks a velocity-servo-driven joint whose limit constraint is active,
+               and whichever jaw hangs below the gripper is pressed into its lower limit by
+               gravity. With the margin, the servo holds q=0 and the limit never engages.
+             - Coulomb friction 5 N > jaw weight (0.129 kg ~ 1.3 N) so an uncontrolled jaw
+               (e.g. before controllers activate) doesn't sag onto the limit either. The 50 N
+               effort budget easily overcomes it when commanded. -->
         <joint name="${prefix}robotiq_85_left_knuckle_joint" type="prismatic">
             <parent link="${prefix}robotiq_85_base_link" />
@@ -215,5 +223,6 @@
             <axis xyz="-1 0 0" />
             <origin xyz="0.03060114 0.0 0.05490452" rpy="0 0 0" />
-            <limit lower="0.0" upper="${robotiq_prismatic_stroke}" effort="50" velocity="0.5" />
+            <limit lower="-0.002" upper="${robotiq_prismatic_stroke}" effort="50" velocity="0.5" />
+            <dynamics damping="1.0" friction="5.0" />
         </joint>
         <joint name="${prefix}robotiq_85_right_knuckle_joint" type="prismatic">
@@ -222,5 +231,6 @@
             <axis xyz="1 0 0" />
             <origin xyz="-0.03060114 0.0 0.05490452" rpy="0 0 0" />
-            <limit lower="0.0" upper="${robotiq_prismatic_stroke}" effort="50" velocity="0.5" />
+            <limit lower="-0.002" upper="${robotiq_prismatic_stroke}" effort="50" velocity="0.5" />
+            <dynamics damping="1.0" friction="5.0" />
         </joint>
     </xacro:macro>
